File: capacitive.kicad_pcb (KiCad board)
At the start: 2 copper layers, 24 x 21.8 mm, 11 parts

Commit message: silkscreen
Other:
- board text added: "Designed by SCU SoftCon Lab"
Changed lines of the file:
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@@
 			)
 			(layer "F.Mask")
-			(net 1)
 		)
 		(fp_arc
@@
 			)
 			(layer "F.Mask")
-			(net 1)
 		)
 		(fp_arc
@@
 			)
 			(layer "F.Mask")
-			(net 1)
 		)
 		(fp_arc
@@
 			)
 			(layer "F.Mask")
-			(net 1)
 		)
 		(fp_poly
@@
 			(fill yes)
 			(layer "F.Mask")
-			(net 1)
 		)
 		(fp_poly
@@
 			(fill yes)
 			(layer "F.Mask")
-			(net 1)
 		)
 		(fp_line
@@
 			)
 			(layer "B.Mask")
-			(net 1)
 		)
 		(fp_arc
@@
 			)
 			(layer "B.Mask")
-			(net 1)
 		)
 		(fp_arc
@@
 			)
 			(layer "B.Mask")
-			(net 1)
 		)
 		(fp_arc
@@
 			)
 			(layer "B.Mask")
-			(net 1)
 		)
 		(fp_arc
@@
 			)
 			(layer "B.Mask")
-			(net 1)
 		)
 		(fp_arc
@@
 			)
 			(layer "B.Mask")
-			(net 1)
 		)
 		(fp_arc
@@
 			)
 			(layer "B.Mask")
-			(net 1)
 		)
 		(fp_arc
@@
 			)
 			(layer "B.Mask")
-			(net 1)
 		)
 		(fp_arc
@@
 			)
 			(layer "B.Mask")
-			(net 1)
 		)
 		(fp_arc
@@
 			)
 			(layer "B.Mask")
-			(net 1)
 		)
 		(fp_arc
@@
 			)
 			(layer "B.Mask")
-			(net 1)
 		)
 		(fp_arc
@@
 			)
 			(layer "B.Mask")
-			(net 1)
 		)
 		(fp_poly
@@
 			(fill yes)
 			(layer "B.Mask")
-			(net 1)
 		)
 		(fp_poly
@@
 			(fill yes)
 			(layer "B.Mask")
-			(net 1)
 		)
 		(fp_text user "${REFERENCE}"
@@
 			)
 			(layer "F.Mask")
-			(net 1)
 		)
 		(fp_arc
@@
 			)
 			(layer "F.Mask")
-			(net 1)
 		)
 		(fp_arc
@@
 			)
 			(layer "F.Mask")
-			(net 1)
 		)
 		(fp_arc
@@
 			)
 			(layer "F.Mask")
-			(net 1)
 		)
 		(fp_poly
@@
 			(fill yes)
 			(layer "F.Mask")
-			(net 1)
 		)
 		(fp_poly
@@
 			(fill yes)
 			(layer "F.Mask")
-			(net 1)
 		)
 		(fp_line
@@
 			)
 			(layer "B.Mask")
-			(net 1)
 		)
 		(fp_arc
@@
 			)
 			(layer "B.Mask")
-			(net 1)
 		)
 		(fp_arc
@@
 			)
 			(layer "B.Mask")
-			(net 1)
 		)
 		(fp_arc
@@
 			)
 			(layer "B.Mask")
-			(net 1)
 		)
 		(fp_arc
@@
 			)
 			(layer "B.Mask")
-			(net 1)
 		)
 		(fp_arc
@@
 			)
 			(layer "B.Mask")
-			(net 1)
 		)
 		(fp_arc
@@
 			)
 			(layer "B.Mask")
-			(net 1)
 		)
 		(fp_arc
@@
 			)
 			(layer "B.Mask")
-			(net 1)
 		)
 		(fp_arc
@@
 			)
 			(layer "B.Mask")
-			(net 1)
 		)
 		(fp_arc
@@
 			)
 			(layer "B.Mask")
-			(net 1)
 		)
 		(fp_arc
@@
 			)
 			(layer "B.Mask")
-			(net 1)
 		)
 		(fp_arc
@@
 			)
 			(layer "B.Mask")
-			(net 1)
 		)
 		(fp_poly
@@
 			(fill yes)
 			(layer "B.Mask")
-			(net 1)
 		)
 		(fp_poly
@@
 			(fill yes)
 			(layer "B.Mask")
-			(net 1)
 		)
 		(fp_text user "${REFERENCE}"
@@
 		(layer "Edge.Cuts")
 	)
+	(gr_text "Designed by \nSCU SoftCon \nLab"
+		(at 142.5 87.75 0)
+		(layer "F.SilkS")
+		(effects
+			(font
+				(size 0.3 0.3)
+				(thickness 0.05)
+				(bold yes)
+			)
+			(justify left bottom)
+		)
+	)
+	(dimension
+		(type orthogonal)
+		(layer "F.SilkS")
+		(pts
+			(xy 140 77.5) (xy 132.75 99.25)
+		)
+		(height 0)
+		(orientation 1)
+		(format
+			(prefix "")
+			(suffix "")
+			(units 3)
+			(units_format 0)
+			(precision 4)
+			(suppress_zeroes yes)
+		)
+		(style
+			(thickness 0.1)
+			(arrow_length 1.27)
+			(text_position_mode 0)
+			(arrow_direction outward)
+			(extension_height 0.58642)
+			(extension_offset 0.5)
+			(keep_text_aligned yes)
+		)
+		(gr_text "21.75"
+			(at 138.9 88.375 90)
+			(layer "F.SilkS")
+			(effects
+				(font
+					(size 1 1)
+					(thickness 0.1)
+				)
+			)
+		)
+	)
 	(segment
